File: TIA/TIA.kicad_sch (KiCad schematic)
At the start: 9 parts, among them J1 Conn_Coaxial, U1 AD8552ARZ

Commit message: added .lck files to .gitignore
Parts:
- added C6: 1.6n, symbol Device:C_Small
- added H2, H3: MountingHole_Pad, MountingHole:MountingHole_3.2mm_M3_Pad_Via, symbol Mechanical:MountingHole_Pad
- added R2: 100, symbol Device:R_Small
- added R3: 10k, symbol Device:R_Small
- added R6: 1k5, symbol Device:R_Small
- C1, C3: footprint (none) -> Capacitor_SMD:C_1206_3216Metric; dist (none) -> Mouser; dist no (none) -> 81-GRM3195C1H104JA5D; man (none) -> Murata; man no (none) -> GRM3195C1H104JA05D
- C2, C4: value 10u -> 4.7u; footprint (none) -> Capacitor_SMD:C_1206_3216Metric; dist (none) -> Mouser; dist no (none) -> 810-C3216X7R1E475K; man (none) -> TDK; man no (none) -> C3216X7R1E475K160AC
Connections:
- net GND: now also U1.3 (+), H2.1, H3.1
- net TIA_IN: now reaches C5.1, H1.1, R1.1, U1.6 (-)
- net TIA_OUT: now reaches C5.2, R1.2, U1.7
- net TIA_OUT: now also R2.2
- net at U1.1: now also C6.1, R3.1, R6.2
- net at U1.2 (-): now also C6.2, R2.1, R3.2
- net at J1.1 (In): now also R6.1
Other:
- moved on the sheet: C1, C5, H1, J1, R1, U1A, U1B
